Commit message: fixed up drive wheel joints, colored body

File: bessie.urdf (robot description, URDF)
Before this commit: robot bessie, 3 links, 2 joints
Links:
- link base_link: geometry collision box size=0.762 0.4572 0.3048; visual box size=0.762 0.4572 0.3048
- link left_wheel: geometry collision cylinder length=0.1016 radius=0.1651; visual cylinder length=0.1016 radius=0.1651
- link right_wheel: geometry collision cylinder length=0.1016 radius=0.1651; visual cylinder length=0.1016 radius=0.1651
Joints:
- joint wheel0: axis (none) -> 1 0 0; origin xyz=0 0 0 rpy=0 0 0 -> xyz=0.2856 0.2922 -0.1131 rpy=0 0 1.5708
- joint wheel1: axis (none) -> 1 0 0; origin xyz=0 0 0 rpy=0 0 0 -> xyz=0.28575 -0.2922 -0.1131 rpy=0 0 -1.5708
