Commit message: added laser frame and link

File: goat.urdf (robot description, URDF)
Before this commit: robot goat, 3 links, 2 joints
Links:
- added link laser; visual cylinder length=0.0349 radius=0.0381
Joints:
- added joint laser_joint: type fixed, parent base_link, child laser, origin xyz=-0.0572 0 0.1715

Commit message: added base_footprint link

File: goat.urdf (robot description, URDF)
Before this commit: robot goat, 4 links, 3 joints
Links:
- added link base_footprint
Joints:
- added joint base_footprint_joint: type fixed, parent base_footprint, child base_link, origin xyz=0 0 0.2814

Commit message: converted into catkin package

File: goat.urdf (robot description, URDF)
Before this commit: robot goat, 5 links, 4 joints
Links:
- added link encoders
Joints:
- added joint encoders_joint: type fixed, parent base_link, child encoders, origin xyz=0.28575 0 -0.1131
