Commit message: moved into urdf/ to install properly, base_link is now tree head

File: urdf/goat.urdf (robot description, URDF)
Before this commit: robot goat, 6 links, 5 joints
Joints:
- joint base_footprint_joint: child base_link -> base_footprint; origin xyz=0 0 0.2814 -> xyz=0 0 -0.2814; parent base_footprint -> base_link

Commit message: Added positioning of encoders, camera, and imu. GPS origin still undefined.

File: urdf/goat.urdf (robot description, URDF)
Before this commit: robot goat, 16 links, 15 joints
Links:
- added link camera; visual box size=0.0381 0.1778 0.0381
- link encoders: geometry visual box size=0.03 0.03 0.03
- link imu: geometry visual box size=0.0508 0.0508 0.025
Joints:
- added joint camera_joint: type fixed, parent base_center, child camera, origin xyz=0.23495 0 0.17145
- joint encoders_joint: origin (none) -> xyz=0.14 0 0; parent base_link -> base_center
- joint imu_joint: origin xyz=0.1922 0 0.1715 rpy=0 0 0 -> xyz=0.0254 0 0.0699 rpy=0 0 0; parent base_center -> top_box

Commit message: moved base_link to be between two encoders

File: urdf/goat.urdf (robot description, URDF)
Before this commit: robot goat, 17 links, 16 joints
Joints:
- joint base_center_joint: origin xyz=0 0 0 -> xyz=-0.14 0 0
