Commit message: added imu joint

File: robots/goat.urdf (robot description, URDF)
Before this commit: robot goat, 6 links, 5 joints
Links:
- added link imu
Joints:
- added joint imu_joint: type fixed, parent base_link, child imu

Commit message: inverted laser frame to reflect clockwise orientation of RPLIDAR A2 scans

File: robots/goat.urdf (robot description, URDF)
Before this commit: robot goat, 7 links, 6 joints
Joints:
- joint laser_joint: origin xyz=-0.0572 0 0.1715 -> xyz=-0.0572 0 0.1715 rpy=3.1416 0 0

Commit message: reversed orientation of RPLIDAR; hector_mapping now simulates properly

File: robots/goat.urdf (robot description, URDF)
Before this commit: robot goat, 7 links, 6 joints
Joints:
- joint laser_joint: origin xyz=-0.0572 0 0.1715 rpy=3.1416 0 0 -> xyz=-0.0572 0 0.1715 rpy=3.1416 0 3.1416

Commit message: corrected laser, imu joint poses

File: robots/goat.urdf (robot description, URDF)
Before this commit: robot goat, 7 links, 6 joints
Joints:
- joint imu_joint: origin (none) -> xyz=0.1922 0 0.1715 rpy=0 0 3.1416
- joint laser_joint: origin xyz=-0.0572 0 0.1715 rpy=3.1416 0 3.1416 -> xyz=0.2032 0 0.2223 rpy=0 0 3.1416

Commit message: moved base_link to between front wheels to increase encoder odometry accuracy, added base_center link where base_link was for convenience

File: robots/goat.urdf (robot description, URDF)
Before this commit: robot goat, 7 links, 6 joints
Links:
- added link base_center; collision box size=0.762 0.4572 0.3048; visual box size=0.762 0.4572 0.3048
- link base_link: geometry 
Joints:
- added joint base_center_joint: type fixed, parent base_link, child base_center, origin xyz=-0.28575 0 0.1131
- joint base_footprint_joint: parent base_link -> base_center
- joint encoders_joint: origin xyz=0.28575 0 -0.1131 -> (none)
- joint imu_joint: parent base_link -> base_center
- joint laser_joint: parent base_link -> base_center
- joint wheel0: parent base_link -> base_center
- joint wheel1: parent base_link -> base_center

Commit message: changed orientation of imu, added gps link

File: robots/goat.urdf (robot description, URDF)
Before this commit: robot goat, 8 links, 7 joints
Links:
- added link gps
Joints:
- added joint gps_joint: type fixed, parent base_center, child gps
- joint imu_joint: origin xyz=0.1922 0 0.1715 rpy=0 0 3.1416 -> xyz=0.1922 0 0.1715 rpy=0 0 0

Commit message: rename urdf->robots, camera->zed_center

File: robots/goat.urdf (robot description, URDF)
Before this commit: robot goat, 17 links, 16 joints
Links:
- removed link camera
- added link zed_center; visual box size=0.0381 0.1778 0.0381
Joints:
- joint camera_joint: child camera -> zed_center
- joint wheel0: origin xyz=0.2 -0.2922 -0.1 rpy=0 0 1.5708 -> xyz=0.2 0.2922 -0.1 rpy=0 0 1.5708
- joint wheel1: origin xyz=0.2 0.2922 -0.1 rpy=0 0 -1.5708 -> xyz=0.2 -0.2922 -0.1 rpy=0 0 -1.5708

Commit message: Added GPS to top of front post

File: robots/goat.urdf (robot description, URDF)
Before this commit: robot goat, 17 links, 16 joints
Links:
- link gps: geometry visual cylinder length=0.0127 radius=0.0254
Joints:
- joint gps_joint: origin (none) -> xyz=0 0 0.26195; parent base_center -> front_post

Commit message: Moved base_link to be between encoders. Moved imu to front of top_box.

File: robots/goat.urdf (robot description, URDF)
Before this commit: robot goat, 17 links, 16 joints
Links:
- link base_link: geometry visual box size=0.01 0.01 0.01
Joints:
- joint base_center_joint: origin xyz=-0.14 0 0 -> xyz=-0.2020 0 0.1
- joint encoders_joint: origin xyz=0.14 0 0 -> xyz=0 0 0; parent base_center -> base_link
- joint imu_joint: origin xyz=0.0254 0 0.0699 rpy=0 0 0 -> xyz=0.126 0 0.0699 rpy=0 0 0

Commit message: adjust imu frame, laser->velodyne frame

File: robots/goat.urdf (robot description, URDF)
Before this commit: robot goat, 17 links, 16 joints
Links:
- removed link laser
- added link velodyne; visual cylinder length=0.0381 radius=0.0381
Joints:
- removed joint laser_joint
- added joint velodyne_joint: type fixed, parent laser_base, child velodyne, origin xyz=0 0 0.0333 rpy=0 0 0
- joint imu_joint: origin xyz=0.126 0 0.0699 rpy=0 0 0 -> xyz=-0.12 0 0.0699 rpy=0 0 3.14159
- joint laser_base_joint: origin xyz=0.0254 0 0.1032 -> xyz=0.07 0 0.1032

Commit message: added an inertial tag to the base link

File: robots/goat.urdf (robot description, URDF)
Before this commit: robot goat, 17 links, 16 joints
Links:
- link base_center: mass None -> 1
- link base_link: mass None -> 1

Commit message: Combine velodyne and robot to the same file

File: robots/goat.urdf (robot description, URDF)
Before this commit: robot goat, 17 links, 16 joints
Links:
- removed link velodyne
- added link goat_velodyne; visual cylinder length=0.0381 radius=0.0381
Joints:
- added joint goat_to_vel: type fixed, parent ex_base_footprint, child base_link, origin xyz=1 1 1 rpy=0 0 0
- joint velodyne_joint: child velodyne -> goat_velodyne

Commit message: linked velodyne to robot model

File: robots/goat.urdf (robot description, URDF)
Before this commit: robot goat, 17 links, 17 joints
Joints:
- joint goat_to_vel: origin xyz=1 1 1 rpy=0 0 0 -> xyz=0 0 0 rpy=0 0 0

File: velodyne/velodyne_description/urdf/example.urdf.xacro (robot description, xacro)
@@ -14,10 +14,10 @@
     <visual>
       <geometry>
-        <box size="0.5 0.5 0.1" />
+        <box size="0.005 0.005 0.001" />
       </geometry>
     </visual>
     <collision>
       <geometry>
-        <box size="0.5 0.5 0.1" />
+        <box size="0.005 0.005 0.001" />
       </geometry>
     </collision>
