Commit message: Pushing working world file to rep

File: world/example.world.xacro (robot description, xacro)
@@ -1,4 +1,3 @@
 <?xml version="1.0" ?>
-<!--<robot xmlns="http://www.ros.org/wiki/xacro" name="world">-->
 <sdf version="1.5">
     <world name="default">
@@ -11,15 +10,13 @@
             <uri>model://ground_plane</uri>
         </include>
-        <!--
-        <xacro:include filename="$(find goat_description)/world/cone.xacro"/>
-        <cone></cone>
-        -->
-        <!-- lets see if this puts a default one in-->
-        <!-- A unit box -->
-        <model name='unit_box_0_0'>
-            <pose frame=''>-1.5 2.5 0.5 0 -0 0</pose>
-            <link name='link'>
-                <inertial>
-                    <mass>1</mass>
+        <!-- start copying and pasting in cones -->
+        <material>
+            <color rgba="249 105 14 1"/>
+        </material>
+        <model name="cone1">
+            <pose frame="cone_frame">2 4 0.5 0 0 0</pose>
+            <link name="main_body">
+                <intertial>
+                    <mass>1</mass> <!-- some sort of default value, does it matter? -->
                     <inertia>
                         <ixx>0.166667</ixx>
@@ -30,17 +27,18 @@
                         <izz>0.166667</izz>
                     </inertia>
-                </inertial>
-                <collision name='collision'>
+                </intertial>
+                <collision name="main_collision">
                     <geometry>
-                        <box>
-                            <size>1 1 1</size>
-                        </box>
+                        <cylinder>
+                            <radius>0.25</radius>
+                            <length>1</length>
+                        </cylinder>
                     </geometry>
-                    <max_contacts>10</max_contacts>
+                    <max_contacts>10</max_contacts><!-- what does this do?-->
                     <surface>
                         <contact>
                             <ode/>
                         </contact>
-                        <bounce/>
+                        <bounce/><!-- what does this do?-->
                         <friction>
                             <torsional>
@@ -53,68 +51,12 @@
                 <visual name='visual'>
                     <geometry>
-                        <box>
-                            <size>1 1 1</size>
-                        </box>
+                        <cylinder>
+                            <radius>0.25</radius>
+                            <length>1</length>
+                        </cylinder>
                     </geometry>
-                    <material>
-                        <script>
-                            <name>Gazebo/Grey</name>
-                            <uri>file://media/materials/scripts/gazebo.material</uri>
-                        </script>
-                    </material>
+                    <material name="orange"/>
                 </visual>
-                <self_collide>0</self_collide>
-                <kinematic>0</kinematic>
-                <gravity>1</gravity>
-            </link>
-        </model>
-        <!-- Another unit box to see if lidar actually works-->
-        <model name='unit_box_0_1'>
-            <pose frame=''>1.3 1.8 0.3 0 0 0</pose>
-            <link name='link'>
-                <inertial>
-                    <mass>1</mass>
-                    <inertia>
-                        <ixx>0.166667</ixx>
-                        <ixy>0</ixy>
-                        <ixz>0</ixz>
-                        <iyy>0.166667</iyy>
-                        <iyz>0</iyz>
-                        <izz>0.166667</izz>
-                    </inertia>
-                </inertial>
-                <collision name='collision'>
-                    <geometry>
-                        <box>
-                            <size>0.5 0.5 0.3</size>
-                        </box>
-                    </geometry>
-                    <max_contacts>10</max_contacts>
-                    <surface>
-                        <contact>
-                            <ode/>
-                        </contact>
-                        <bounce/>
-                        <friction>
-                            <torsional>
-                                <ode/>
-                            </torsional>
-                            <ode/>
-                        </friction>
-                    </surface>
-                </collision>
-                <visual name='visual'>
-                    <geometry>
-                        <box>
-                            <size>0.5 0.5 0.3</size>
-                        </box>
-                    </geometry>
-                    <material>
-                        <script>
-                            <name>Gazebo/Grey</name>
-                            <uri>file://media/materials/scripts/gazebo.material</uri>
-                        </script>
-                    </material>
-                </visual>
+                <!-- don't know what these 3 things do -->
                 <self_collide>0</self_collide>
                 <kinematic>0</kinematic>
@@ -124,3 +66,2 @@
     </world>
 </sdf>
-<!--</robot>-->
